File: board/try two.brd (EAGLE design)
At the start: 94.9 x 78.7 mm, 19 parts

Commit message: Better routing
Parts:
- moved WIZJ2 72.9 mm to (10.2, 72.4), turned to 180 degrees
- moved PH1 5.08 mm to (34.3, 55.9)
- moved PH2 5.08 mm to (34.3, 41.9)
- moved PH3 5.08 mm to (34.3, 26.7)
- moved PH7 5.08 mm to (33.0, 55.9)
- moved PH8 5.08 mm to (33.0, 41.9)
- moved PH9 5.08 mm to (33.0, 26.7)
- moved PH10 1.27 mm to (71.1, 55.9)
- moved PH11 1.27 mm to (71.1, 41.9)
- moved PH12 1.27 mm to (71.1, 27.9)
- moved PH4 1.27 mm to (69.8, 55.9)
- moved PH5 1.27 mm to (69.8, 41.9)
- moved PH6 1.27 mm to (69.8, 27.9)
Connections:
- removed net N$10: PH9.3
- net INTC: now also PH9.3
Routing:
- net INTC: track 0.00 -> 38.7 mm, vias 0 -> 1
- net CSA: track 0.00 -> 37.1 mm, vias 0 -> 2
- net SDI: track 178.3 -> 149.3 mm, vias 2 -> 3
- net SCLK: track 130.0 -> 149.6 mm
- net CSB: track 13.5 -> 25.1 mm
- net GND: track 152.4 -> 161.9 mm, vias 3 -> 4
- net INTB: track 15.6 -> 24.8 mm
- net ECL: track 117.5 -> 123.7 mm, vias 1 -> 4
- net CSC: track 65.6 -> 71.6 mm
- net EDA: track 108.8 -> 114.6 mm
- net CSD: track 33.5 -> 37.4 mm
- net SD0: track 175.9 -> 173.2 mm, vias 4 -> 1
- net INTA: track 17.7 -> 19.9 mm
- net INTF: track 13.9 -> 15.9 mm
- net VCC3: track 172.6 -> 170.9 mm, vias 0 -> 1
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