File: board/try two.sch (EAGLE design)
At the start: 19 parts

Commit message: Better routing
Connections:
- removed net N$10: PH9.3
- net INTC: now also PH9.3
Changed lines of the file:
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@@
-</segment>
-</net>
-<net name="INTC" class="0">
-<segment>
-<pinref part="T-2" gate="G$1" pin="7"/>
-<label x="-5.08" y="149.86" size="1.778" layer="95" xref="yes"/>
-<wire x1="48.26" y1="147.32" x2="40.64" y2="147.32" width="0.1524" layer="91"/>
-<wire x1="40.64" y1="147.32" x2="40.64" y2="149.86" width="0.1524" layer="91"/>
-<wire x1="40.64" y1="149.86" x2="-20.32" y2="149.86" width="0.1524" layer="91"/>
 </segment>
 </net>
@@
 </segment>
 </net>
-<net name="N$10" class="0">
-<segment>
-<pinref part="PH9" gate="G$1" pin="3"/>
-<wire x1="71.12" y1="147.32" x2="48.26" y2="147.32" width="0.1524" layer="91"/>
-</segment>
-</net>
 <net name="N$12" class="0">
 <segment>
@@
 </segment>
 </net>
+<net name="INTC" class="0">
+<segment>
+<pinref part="T-2" gate="G$1" pin="7"/>
+<wire x1="-20.32" y1="149.86" x2="45.72" y2="149.86" width="0.1524" layer="91"/>
+<wire x1="45.72" y1="149.86" x2="45.72" y2="147.32" width="0.1524" layer="91"/>
+<pinref part="PH9" gate="G$1" pin="3"/>
+<wire x1="45.72" y1="147.32" x2="71.12" y2="147.32" width="0.1524" layer="91"/>
+<label x="45.72" y="152.4" size="1.778" layer="95"/>
+</segment>
+</net>
